File: test_pcbs/test_pcb.kicad_pcb (KiCad board)
At the start: 2 copper layers, 36.6 x 26.5 mm, 6 parts

Commit message: Code refactor
Parts:
- R3, R4: footprint Resistor_SMD:R_1812_4532Metric_Pad1.30x3.40mm_HandSolder -> Capacitor_SMD:C_1812_4532Metric
Changed lines of the file:
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@@
     )
   )
-  (footprint "Resistor_SMD:R_1812_4532Metric_Pad1.30x3.40mm_HandSolder" (layer "B.Cu")
+  (footprint "Capacitor_SMD:C_1812_4532Metric" (layer "B.Cu")
     (at 124.33 81.28 180)
-    (descr "Resistor SMD 1812 (4532 Metric), square (rectangular) end terminal, IPC_7351 nominal with elongated pad for handsoldering. (Body size source: https://www.nikhef.nl/pub/departments/mt/projects/detectorR_D/dtddice/ERJ2G.pdf), generated with kicad-footprint-generator")
-    (tags "resistor handsolder")
+    (descr "Capacitor SMD 1812 (4532 Metric), square (rectangular) end terminal, IPC_7351 nominal, (Body size source: IPC-SM-782 page 76, https://www.pcb-3d.com/wordpress/wp-content/uploads/ipc-sm-782a_amendment_1_and_2.pdf), generated with kicad-footprint-generator")
+    (tags "capacitor")
     (property "Sheetfile" "test_pcb.kicad_sch")
     (property "Sheetname" "")
@@
         (effects (font (size 1 1) (thickness 0.15)) (justify mirror))
     )
-    (fp_line (start -1.386252 -1.71) (end 1.386252 -1.71)
+    (fp_line (start -1.161252 -1.71) (end 1.161252 -1.71)
       (stroke (width 0.12) (type solid)) (layer "B.SilkS"))
-    (fp_line (start -1.386252 1.71) (end 1.386252 1.71)
+    (fp_line (start -1.161252 1.71) (end 1.161252 1.71)
       (stroke (width 0.12) (type solid)) (layer "B.SilkS"))
-    (fp_line (start -3.12 -1.95) (end -3.12 1.95)
+    (fp_line (start -3 -1.95) (end -3 1.95)
       (stroke (width 0.05) (type solid)) (layer "B.CrtYd"))
-    (fp_line (start -3.12 1.95) (end 3.12 1.95)
+    (fp_line (start -3 1.95) (end 3 1.95)
       (stroke (width 0.05) (type solid)) (layer "B.CrtYd"))
-    (fp_line (start 3.12 -1.95) (end -3.12 -1.95)
+    (fp_line (start 3 -1.95) (end -3 -1.95)
       (stroke (width 0.05) (type solid)) (layer "B.CrtYd"))
-    (fp_line (start 3.12 1.95) (end 3.12 -1.95)
+    (fp_line (start 3 1.95) (end 3 -1.95)
       (stroke (width 0.05) (type solid)) (layer "B.CrtYd"))
     (fp_line (start -2.25 -1.6) (end -2.25 1.6)
@@
     (fp_line (start 2.25 1.6) (end 2.25 -1.6)
       (stroke (width 0.1) (type solid)) (layer "B.Fab"))
-    (pad "1" smd roundrect (at -2.225 0 180) (size 1.3 3.4) (layers "B.Cu" "B.Paste" "B.Mask") (roundrect_rratio 0.192308)
+    (pad "1" smd roundrect (at -2.05 0 180) (size 1.4 3.4) (layers "B.Cu" "B.Paste" "B.Mask") (roundrect_rratio 0.178571)
       (net 6 "Net-(R3-Pad2)") (pintype "passive"))
-    (pad "2" smd roundrect (at 2.225 0 180) (size 1.3 3.4) (layers "B.Cu" "B.Paste" "B.Mask") (roundrect_rratio 0.192308)
+    (pad "2" smd roundrect (at 2.05 0 180) (size 1.4 3.4) (layers "B.Cu" "B.Paste" "B.Mask") (roundrect_rratio 0.178571)
       (net 1 "Net-(D1-K)") (pintype "passive"))
-    (model "${KICAD6_3DMODEL_DIR}/Resistor_SMD.3dshapes/R_1812_4532Metric.wrl"
+    (model "${KICAD6_3DMODEL_DIR}/Capacitor_SMD.3dshapes/C_1812_4532Metric.wrl"
       (offset (xyz 0 0 0))
       (scale (xyz 1 1 1))
@@
     )
   )
-  (footprint "Resistor_SMD:R_1812_4532Metric_Pad1.30x3.40mm_HandSolder" (layer "B.Cu")
+  (footprint "Capacitor_SMD:C_1812_4532Metric" (layer "B.Cu")
     (at 117.33 81.28 180)
-    (descr "Resistor SMD 1812 (4532 Metric), square (rectangular) end terminal, IPC_7351 nominal with elongated pad for handsoldering. (Body size source: https://www.nikhef.nl/pub/departments/mt/projects/detectorR_D/dtddice/ERJ2G.pdf), generated with kicad-footprint-generator")
-    (tags "resistor handsolder")
+    (descr "Capacitor SMD 1812 (4532 Metric), square (rectangular) end terminal, IPC_7351 nominal, (Body size source: IPC-SM-782 page 76, https://www.pcb-3d.com/wordpress/wp-content/uploads/ipc-sm-782a_amendment_1_and_2.pdf), generated with kicad-footprint-generator")
+    (tags "capacitor")
     (property "Sheetfile" "test_pcb.kicad_sch")
     (property "Sheetname" "")
@@
         (effects (font (size 1 1) (thickness 0.15)) (justify mirror))
     )
-    (fp_line (start -1.386252 -1.71) (end 1.386252 -1.71)
+    (fp_line (start -1.161252 -1.71) (end 1.161252 -1.71)
       (stroke (width 0.12) (type solid)) (layer "B.SilkS"))
-    (fp_line (start -1.386252 1.71) (end 1.386252 1.71)
+    (fp_line (start -1.161252 1.71) (end 1.161252 1.71)
       (stroke (width 0.12) (type solid)) (layer "B.SilkS"))
-    (fp_line (start -3.12 -1.95) (end -3.12 1.95)
+    (fp_line (start -3 -1.95) (end -3 1.95)
       (stroke (width 0.05) (type solid)) (layer "B.CrtYd"))
-    (fp_line (start -3.12 1.95) (end 3.12 1.95)
+    (fp_line (start -3 1.95) (end 3 1.95)
       (stroke (width 0.05) (type solid)) (layer "B.CrtYd"))
-    (fp_line (start 3.12 -1.95) (end -3.12 -1.95)
+    (fp_line (start 3 -1.95) (end -3 -1.95)
       (stroke (width 0.05) (type solid)) (layer "B.CrtYd"))
-    (fp_line (start 3.12 1.95) (end 3.12 -1.95)
+    (fp_line (start 3 1.95) (end 3 -1.95)
       (stroke (width 0.05) (type solid)) (layer "B.CrtYd"))
     (fp_line (start -2.25 -1.6) (end -2.25 1.6)
@@
     (fp_line (start 2.25 1.6) (end 2.25 -1.6)
       (stroke (width 0.1) (type solid)) (layer "B.Fab"))
-    (pad "1" smd roundrect (at -2.225 0 180) (size 1.3 3.4) (layers "B.Cu" "B.Paste" "B.Mask") (roundrect_rratio 0.192308)
+    (pad "1" smd roundrect (at -2.05 0 180) (size 1.4 3.4) (layers "B.Cu" "B.Paste" "B.Mask") (roundrect_rratio 0.178571)
       (net 5 "Net-(BT1--)") (pintype "passive"))
-    (pad "2" smd roundrect (at 2.225 0 180) (size 1.3 3.4) (layers "B.Cu" "B.Paste" "B.Mask") (roundrect_rratio 0.192308)
+    (pad "2" smd roundrect (at 2.05 0 180) (size 1.4 3.4) (layers "B.Cu" "B.Paste" "B.Mask") (roundrect_rratio 0.178571)
       (net 6 "Net-(R3-Pad2)") (pintype "passive"))
-    (model "${KICAD6_3DMODEL_DIR}/Resistor_SMD.3dshapes/R_1812_4532Metric.wrl"
+    (model "${KICAD6_3DMODEL_DIR}/Capacitor_SMD.3dshapes/C_1812_4532Metric.wrl"
       (offset (xyz 0 0 0))
       (scale (xyz 1 1 1))

Commit message: import statement
Parts:
- moved D1 2.54 mm to (132.1, 76.2)
Changed lines of the file:
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@@
   )
   (footprint "LED_THT:LED_D5.0mm" (layer "F.Cu")
-    (at 132.08 73.66 -90)
+    (at 132.08 76.2 -90)
     (descr "LED, diameter 5.0mm, 2 pins, http://cdn-reichelt.de/documents/datenblatt/A500/LL-504BC2E-009.pdf")
     (tags "LED diameter 5.0mm 2 pins")
